Commit message: Fix MG400 Cartesian IK across J1 branch boundary
- add robot-specific IK post-processing hook
- enforce MG400 parallel-link joint coupling
- unwrap J1 targets relative to the current angle
- widen MG400 J1 limits to ±2π across all URDF vari

File: tactile_sim/assets/embodiment_assets/combined_urdfs/mg400_flat_tactip.urdf (robot description, URDF)
Before this commit: robot mg400, 14 links, 13 joints
Joints:
- joint j1: limit lower=-3.14000 upper=3.14000 effort=0.00000 velocity=0.00000 -> lower=-6.28319 upper=6.28319 effort=0.00000 velocity=0.00000

File: tactile_sim/assets/embodiment_assets/combined_urdfs/mg400_mini_tactip.urdf (robot description, URDF)
Before this commit: robot mg400, 14 links, 13 joints
Joints:
- joint j1: limit lower=-3.14000 upper=3.14000 effort=0.00000 velocity=0.00000 -> lower=-6.28319 upper=6.28319 effort=0.00000 velocity=0.00000

File: tactile_sim/assets/embodiment_assets/combined_urdfs/mg400_right_angle_digit.urdf (robot description, URDF)
Before this commit: robot mg400, 14 links, 13 joints
Joints:
- joint j1: limit lower=-3.14000 upper=3.14000 effort=0.00000 velocity=0.00000 -> lower=-6.28319 upper=6.28319 effort=0.00000 velocity=0.00000

File: tactile_sim/assets/embodiment_assets/combined_urdfs/mg400_right_angle_digitac.urdf (robot description, URDF)
Before this commit: robot mg400, 14 links, 13 joints
Joints:
- joint j1: limit lower=-3.14000 upper=3.14000 effort=0.00000 velocity=0.00000 -> lower=-6.28319 upper=6.28319 effort=0.00000 velocity=0.00000

File: tactile_sim/assets/embodiment_assets/combined_urdfs/mg400_right_angle_tactip.urdf (robot description, URDF)
Before this commit: robot mg400, 15 links, 14 joints
Joints:
- joint j1: limit lower=-3.14000 upper=3.14000 effort=0.00000 velocity=0.00000 -> lower=-6.28319 upper=6.28319 effort=0.00000 velocity=0.00000

File: tactile_sim/assets/embodiment_assets/combined_urdfs/mg400_standard_digit.urdf (robot description, URDF)
Before this commit: robot mg400, 14 links, 13 joints
Joints:
- joint j1: limit lower=-3.14000 upper=3.14000 effort=0.00000 velocity=0.00000 -> lower=-6.28319 upper=6.28319 effort=0.00000 velocity=0.00000

File: tactile_sim/assets/embodiment_assets/combined_urdfs/mg400_standard_digitac.urdf (robot description, URDF)
Before this commit: robot mg400, 14 links, 13 joints
Joints:
- joint j1: limit lower=-3.14000 upper=3.14000 effort=0.00000 velocity=0.00000 -> lower=-6.28319 upper=6.28319 effort=0.00000 velocity=0.00000

File: tactile_sim/assets/embodiment_assets/combined_urdfs/mg400_standard_tactip.urdf (robot description, URDF)
Before this commit: robot mg400, 14 links, 13 joints
Joints:
- joint j1: limit lower=-3.14000 upper=3.14000 effort=0.00000 velocity=0.00000 -> lower=-6.28319 upper=6.28319 effort=0.00000 velocity=0.00000

File: tactile_sim/assets/robot_arm_assets/mg400/urdfs/mg400.urdf (robot description, URDF)
Before this commit: robot mg400, 11 links, 10 joints
Joints:
- joint j1: limit lower=-3.14 upper=3.14 effort=0 velocity=0 -> lower=-6.28319 upper=6.28319 effort=0 velocity=0

Commit message: Fix MG400 coupled joint limits and movement diagnostics
Expand the MG400 j5 and j4_2 limits to ±2π across the source and
combined embodiment URDFs. Validate coupled IK targets against URDF
joint limits and report per-joint errors when blocking moves time out.

File: tactile_sim/assets/embodiment_assets/combined_urdfs/mg400_flat_tactip.urdf (robot description, URDF)
Before this commit: robot mg400, 14 links, 13 joints
Joints:
- joint j4_2: limit lower=-3.14000 upper=3.14000 effort=0.00000 velocity=0.00000 -> lower=-6.28319 upper=6.28319 effort=0.00000 velocity=0.00000
- joint j5: limit lower=-3.14000 upper=3.14000 effort=0.00000 velocity=0.00000 -> lower=-6.28319 upper=6.28319 effort=0.00000 velocity=0.00000

File: tactile_sim/assets/embodiment_assets/combined_urdfs/mg400_mini_tactip.urdf (robot description, URDF)
Before this commit: robot mg400, 14 links, 13 joints
Joints:
- joint j4_2: limit lower=-3.14000 upper=3.14000 effort=0.00000 velocity=0.00000 -> lower=-6.28319 upper=6.28319 effort=0.00000 velocity=0.00000
- joint j5: limit lower=-3.14000 upper=3.14000 effort=0.00000 velocity=0.00000 -> lower=-6.28319 upper=6.28319 effort=0.00000 velocity=0.00000

File: tactile_sim/assets/embodiment_assets/combined_urdfs/mg400_right_angle_digit.urdf (robot description, URDF)
Before this commit: robot mg400, 14 links, 13 joints
Joints:
- joint j4_2: limit lower=-3.14000 upper=3.14000 effort=0.00000 velocity=0.00000 -> lower=-6.28319 upper=6.28319 effort=0.00000 velocity=0.00000
- joint j5: limit lower=-3.14000 upper=3.14000 effort=0.00000 velocity=0.00000 -> lower=-6.28319 upper=6.28319 effort=0.00000 velocity=0.00000

File: tactile_sim/assets/embodiment_assets/combined_urdfs/mg400_right_angle_digitac.urdf (robot description, URDF)
Before this commit: robot mg400, 14 links, 13 joints
Joints:
- joint j4_2: limit lower=-3.14000 upper=3.14000 effort=0.00000 velocity=0.00000 -> lower=-6.28319 upper=6.28319 effort=0.00000 velocity=0.00000
- joint j5: limit lower=-3.14000 upper=3.14000 effort=0.00000 velocity=0.00000 -> lower=-6.28319 upper=6.28319 effort=0.00000 velocity=0.00000

File: tactile_sim/assets/embodiment_assets/combined_urdfs/mg400_right_angle_tactip.urdf (robot description, URDF)
Before this commit: robot mg400, 15 links, 14 joints
Joints:
- joint j4_2: limit lower=-3.14000 upper=3.14000 effort=0.00000 velocity=0.00000 -> lower=-6.28319 upper=6.28319 effort=0.00000 velocity=0.00000
- joint j5: limit lower=-3.14000 upper=3.14000 effort=0.00000 velocity=0.00000 -> lower=-6.28319 upper=6.28319 effort=0.00000 velocity=0.00000

File: tactile_sim/assets/embodiment_assets/combined_urdfs/mg400_standard_digit.urdf (robot description, URDF)
Before this commit: robot mg400, 14 links, 13 joints
Joints:
- joint j4_2: limit lower=-3.14000 upper=3.14000 effort=0.00000 velocity=0.00000 -> lower=-6.28319 upper=6.28319 effort=0.00000 velocity=0.00000
- joint j5: limit lower=-3.14000 upper=3.14000 effort=0.00000 velocity=0.00000 -> lower=-6.28319 upper=6.28319 effort=0.00000 velocity=0.00000

File: tactile_sim/assets/embodiment_assets/combined_urdfs/mg400_standard_digitac.urdf (robot description, URDF)
Before this commit: robot mg400, 14 links, 13 joints
Joints:
- joint j4_2: limit lower=-3.14000 upper=3.14000 effort=0.00000 velocity=0.00000 -> lower=-6.28319 upper=6.28319 effort=0.00000 velocity=0.00000
- joint j5: limit lower=-3.14000 upper=3.14000 effort=0.00000 velocity=0.00000 -> lower=-6.28319 upper=6.28319 effort=0.00000 velocity=0.00000

File: tactile_sim/assets/embodiment_assets/combined_urdfs/mg400_standard_tactip.urdf (robot description, URDF)
Before this commit: robot mg400, 14 links, 13 joints
Joints:
- joint j4_2: limit lower=-3.14000 upper=3.14000 effort=0.00000 velocity=0.00000 -> lower=-6.28319 upper=6.28319 effort=0.00000 velocity=0.00000
- joint j5: limit lower=-3.14000 upper=3.14000 effort=0.00000 velocity=0.00000 -> lower=-6.28319 upper=6.28319 effort=0.00000 velocity=0.00000

File: tactile_sim/assets/robot_arm_assets/mg400/urdfs/mg400.urdf (robot description, URDF)
Before this commit: robot mg400, 11 links, 10 joints
Joints:
- joint j4_2: limit lower=-3.14 upper=3.14 effort=0 velocity=0 -> lower=-6.28319 upper=6.28319 effort=0 velocity=0
- joint j5: limit lower=-3.14 upper=3.14 effort=0 velocity=0 -> lower=-6.28319 upper=6.28319 effort=0 velocity=0
